Commit message: make naming consistent for cr45

File: urdf/cr45.urdf (robot description, URDF)
Before this commit: robot robot, 8 links, 7 joints
Links:
- link base_link: geometry collision mesh filename=package://rokae_description/meshes/cr45/base_link.obj; visual mesh filename=package://rokae_description/meshes/cr45/base_link.obj
- link link_1: geometry collision mesh filename=package://rokae_description/meshes/cr45/link_1.obj; visual mesh filename=package://rokae_description/meshes/cr45/link_1.obj
- link link_2: geometry collision mesh filename=package://rokae_description/meshes/cr45/link_2.obj; visual mesh filename=package://rokae_description/meshes/cr45/link_2.obj
- link link_3: geometry collision mesh filename=package://rokae_description/meshes/cr45/link_3.obj; visual mesh filename=package://rokae_description/meshes/cr45/link_3.obj
- link link_4: geometry collision mesh filename=package://rokae_description/meshes/cr45/link_4.obj; visual mesh filename=package://rokae_description/meshes/cr45/link_4.obj
- link link_5: geometry collision mesh filename=package://rokae_description/meshes/cr45/link_5.obj; visual mesh filename=package://rokae_description/meshes/cr45/link_5.obj
- link link_6: geometry collision mesh filename=package://rokae_description/meshes/cr45/link_6.obj; visual mesh filename=package://rokae_description/meshes/cr45/link_6.obj
